File: pedal-breakout-pcb.kicad_pcb (KiCad board)
At the start: 2 copper layers, 35 x 175 mm, 30 parts

Commit message: version2 files
Parts:
- removed H2: MountingHole, MountingHole:MountingHole_3.2mm_M3_Pad_Via
- removed LOGO4: **REF, ct-kicad:pedalinator-qr-10mm
- added H4: MountingHole, MountingHole:MountingHole_5mm, F.Cu at (26.5, 27.5)
- added H5: MountingHole, MountingHole:MountingHole_5mm, F.Cu at (51.5, 27.5)
- JB0, JB1, JB2, JB3, JB4, JB5, JB6, JB7, JSRC0, JSRC1, JSRC2: footprint Connector_PinSocket_2.54mm:PinSocket_1x06_P2.54mm_Vertical -> Connector_JST:JST_XH_1x06_P2.50mm_Horizontal-CT
- JEX0: footprint Connector_PinSocket_2.54mm:PinSocket_1x08_P2.54mm_Vertical -> Connector_JST:JST_XH_1x08_P2.50mm_Horizontal-CT
- JIN0, JIN1, JIN2, JIN3, JIN4, JIN5, JIN6, JIN7, JIN8: footprint Connector_PinSocket_2.54mm:PinSocket_1x04_P2.54mm_Vertical -> Connector_JST:JST_XH_1x04_P2.50mm_Horizontal-CT
- JRST0: footprint Connector_PinSocket_2.54mm:PinSocket_1x02_P2.54mm_Vertical -> Connector_JST:JST_XH_S2B-XH-A_1x02_P2.50mm_Horizontal
- LOGO1, LOGO3: moved to F.Cu
- LOGO2: moved to B.Cu
- moved JEX0 198.2 mm to (30.2, 206.5), turned to 0 degrees
- moved JRST0 175.0 mm to (54.2, 197.0), turned to -90 degrees
- moved H1 149.7 mm to (39.0, 177.5)
- moved JB6 111.6 mm to (23.5, 142.0), turned to 90 degrees
- moved JB0 108.8 mm to (23.5, 68.0), turned to 90 degrees
- moved JB2 108.8 mm to (23.5, 86.5), turned to 90 degrees
- moved JIN2 108.8 mm to (23.5, 155.5), turned to 90 degrees
- moved JIN4 108.8 mm to (23.5, 169.0), turned to 90 degrees
- moved JIN6 108.8 mm to (23.5, 182.5), turned to 90 degrees
- moved JIN8 108.8 mm to (23.5, 196.0), turned to 90 degrees
- moved H3 98.8 mm to (39.0, 52.5)
- moved JTX0 88.9 mm to (41.2, 18.0)
- moved LOGO2 87.1 mm to (38.6, 95.8)
- moved LOGO1 87.1 mm to (39.0, 169.7)
- moved JB3 80.8 mm to (23.5, 105.0), turned to 90 degrees
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Connections:
- JB0 pad 1: Net-(JB0-Pin_1) -> GND
- JB0 pad 2: LED-SIG -> +5V
- JB0 pad 3: COL0 -> ROW0
- JB0 pad 4: ROW0 -> COL0
- JB0 pad 5: +5V -> LED-SIG
- JB0 pad 6: GND -> Net-(JB0-Pin_6)
- JB1 pad 1: Net-(JB1-Pin_1) -> GND
- JB1 pad 2: Net-(JB0-Pin_1) -> +5V
- JB1 pad 3: COL1 -> ROW0
- JB1 pad 4: ROW0 -> COL1
- JB1 pad 5: +5V -> Net-(JB0-Pin_6)
- JB1 pad 6: GND -> Net-(JB1-Pin_6)
- JB2 pad 1: Net-(JB2-Pin_1) -> GND
- JB2 pad 2: Net-(JB1-Pin_1) -> +5V
- JB2 pad 3: COL2 -> ROW0
- JB2 pad 4: ROW0 -> COL2
- JB2 pad 5: +5V -> Net-(JB1-Pin_6)
- JB2 pad 6: GND -> Net-(JB2-Pin_6)
- JB3 pad 1: Net-(JB3-Pin_1) -> GND
- JB3 pad 2: Net-(JB2-Pin_1) -> +5V
- JB3 pad 3: COL3 -> ROW0
- JB3 pad 4: ROW0 -> COL3
- JB3 pad 5: +5V -> Net-(JB2-Pin_6)
- JB3 pad 6: GND -> Net-(JB3-Pin_6)
- JB4 pad 1: Net-(JB4-Pin_1) -> GND
- JB4 pad 2: Net-(JB3-Pin_1) -> +5V
- JB4 pad 3: COL0 -> ROW1
- JB4 pad 4: ROW1 -> COL0
- JB4 pad 5: +5V -> Net-(JB3-Pin_6)
- JB4 pad 6: GND -> Net-(JB4-Pin_6)
- JB5 pad 1: Net-(JB5-Pin_1) -> GND
- JB5 pad 2: Net-(JB4-Pin_1) -> +5V
- JB5 pad 3: COL1 -> ROW1
- JB5 pad 4: ROW1 -> COL1
- JB5 pad 5: +5V -> Net-(JB4-Pin_6)
- JB5 pad 6: GND -> Net-(JB5-Pin_6)
- JB6 pad 1: Net-(JB6-Pin_1) -> GND
- JB6 pad 2: Net-(JB5-Pin_1) -> +5V
- JB6 pad 3: COL2 -> ROW1
- JB6 pad 4: ROW1 -> COL2
- JB6 pad 5: +5V -> Net-(JB5-Pin_6)
- JB6 pad 6: GND -> Net-(JB6-Pin_6)
- JB7 pad 1: LED-INT-IND -> GND
- JB7 pad 2: Net-(JB6-Pin_1) -> +5V
- JB7 pad 3: COL3 -> ROW1
- JB7 pad 4: ROW1 -> COL3
- JB7 pad 5: +5V -> Net-(JB6-Pin_6)
- JB7 pad 6: GND -> LED-INT-IND
- JRST0 pad 1: RESET -> GND
- JRST0 pad 2: GND -> RESET
- JSRC0 pad 1: ROW1 -> GND
- JSRC0 pad 2: ROW0 -> +5V
- JSRC0 pad 5: +5V -> ROW0
- JSRC0 pad 6: GND -> ROW1
Routing:
- net LED-IND: track 184.9 -> 32.0 mm, vias 3 -> 2
- net RESET: track 54.5 -> 196.8 mm, vias 0 -> 10
- net ROW0: track 138.6 -> 245.9 mm, vias 10 -> 14
- net COL4: track 49.7 -> 152.4 mm, vias 1 -> 6
- net ROW1: track 181.4 -> 250.2 mm, vias 10 -> 15
- net Net-(JB0-Pin_6): track 0.00 -> 57.2 mm, vias 0 -> 6
- net Net-(JB6-Pin_6): track 0.00 -> 46.8 mm
- net Net-(JB4-Pin_6): track 0.00 -> 46.7 mm, vias 0 -> 2
- net Net-(JB5-Pin_1): track 46.7 -> 0.00 mm, vias 4 -> 0
- net Net-(JB3-Pin_1): track 45.0 -> 0.00 mm, vias 4 -> 0
- net Net-(JB6-Pin_1): track 44.8 -> 0.00 mm, vias 4 -> 0
- net Net-(JB2-Pin_1): track 42.9 -> 0.00 mm, vias 4 -> 0
- net Net-(JB0-Pin_1): track 42.6 -> 0.00 mm, vias 4 -> 0
- net Net-(JB4-Pin_1): track 42.4 -> 0.00 mm, vias 4 -> 0
- net Net-(JB2-Pin_6): track 0.00 -> 40.1 mm, vias 0 -> 2
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Other:
- board size 35 x 175 mm -> 38 x 190 mm
- board text added: "125mm center"
- board text added: "B1"
- board text added: "B2"
- board text added: "B3"
- board text added: "B4"
- board text added: "B5"
- board text added: "B6"
- board text added: "B7"
- board text added: "B8"
- board text added: "BUTTONS"
- board text added: "C4"
- board text added: "COL4"
- board text added: "COM COLS"
- board text added: "DO DI 5V GD"
- board text added: "DO DI C0 R0 5V GD"
- board text added: "DO DI C1 R1 5V GD"
- board text added: "DO DI C2 R0 5V GD"
- board text added: "DO DI C2 R1 5V GD"
- board text added: "DO DI C3 R0 5V GD"
- board text added: "EXT-INDICATOR"
- board text added: "EXT-LED-DI"
- board text added: "FOOT-INATOR"
- board text added: "GD 5V DI C4 R0 R1 RS"
- board text added: "GD 5V DI DO"
- board text added: "GD 5V R0 C1 DI DO"
- board text added: "GD 5V R1 C0 DI DO"
- board text added: "GD 5V R1 C3 DI DO"
- board text added: "LED-1"
- board text added: "LED-2"
- board text added: "LED-3"
- board text added: "LED-4"
- board text added: "LED-5"
- board text added: "LED-6"
- board text added: "LED-7"
- board text added: "LED-8"
- board text added: "LED-9"
- board text added: "LED-EXT"
- board text added: "LEDS"
- board text added: "MCU"
- board text added: "PWR DI RWS"
- board text added: "R1 R0 DI RS 5V GD"
- board text added: "RESET"
- board text added: "SERIAL"
- board text added: "TRRS Soldering fixture 25mm center 5mm holes"
- board text added: "TX RX C3 C2 C1 C0"
- board text added: "v2.0"
- board text removed: "Footinator"
- board text removed: "v1.0"
