File: pedal-breakout-pcb.kicad_sch (KiCad schematic)
At the start: 30 parts

Commit message: version2 files
Parts:
- removed H2: MountingHole, MountingHole:MountingHole_3.2mm_M3_Pad_Via, symbol Mechanical:MountingHole
- removed LOGO4: **REF, ct-kicad:pedalinator-qr-10mm, symbol ct-kicad:pedalinator-qr-10mm
- added H4, H5: MountingHole, MountingHole:MountingHole_5mm, symbol Mechanical:MountingHole
- JB0, JB1, JB2, JB3, JB4, JB5, JB6, JB7, JSRC0, JSRC1, JSRC2: footprint Connector_PinSocket_2.54mm:PinSocket_1x06_P2.54mm_Vertical -> Connector_JST:JST_XH_1x06_P2.50mm_Horizontal-CT
- JEX0: footprint Connector_PinSocket_2.54mm:PinSocket_1x08_P2.54mm_Vertical -> Connector_JST:JST_XH_1x08_P2.50mm_Horizontal-CT
- JIN0, JIN1, JIN2, JIN3, JIN4, JIN5, JIN6, JIN7, JIN8: footprint Connector_PinSocket_2.54mm:PinSocket_1x04_P2.54mm_Vertical -> Connector_JST:JST_XH_1x04_P2.50mm_Horizontal-CT
- JRST0: footprint Connector_PinSocket_2.54mm:PinSocket_1x02_P2.54mm_Vertical -> Connector_JST:JST_XH_S2B-XH-A_1x02_P2.50mm_Horizontal
Connections:
- net +5V: now also JB0.2 (Pin_2), JB1.2 (Pin_2), JB2.2 (Pin_2), JB3.2 (Pin_2), JB4.2 (Pin_2), JB5.2 (Pin_2), JB6.2 (Pin_2), JB7.2 (Pin_2), JSRC0.2 (Pin_2); no longer JB0.5 (Pin_5), JB1.5 (Pin_5), JB2.5 (Pin_5), JB3.5 (Pin_5), JB4.5 (Pin_5), JB5.5 (Pin_5), JB6.5 (Pin_5), JB7.5 (Pin_5), JSRC0.5 (Pin_5)
- net COL0: now also JB0.4 (Pin_4), JB4.4 (Pin_4); no longer JB0.3 (Pin_3), JB4.3 (Pin_3)
- net COL1: now also JB1.4 (Pin_4), JB5.4 (Pin_4); no longer JB1.3 (Pin_3), JB5.3 (Pin_3)
- net COL2: now also JB2.4 (Pin_4), JB6.4 (Pin_4); no longer JB2.3 (Pin_3), JB6.3 (Pin_3)
- net COL3: now also JB3.4 (Pin_4), JB7.4 (Pin_4); no longer JB3.3 (Pin_3), JB7.3 (Pin_3)
- net GND: now also JB0.1 (Pin_1), JB1.1 (Pin_1), JB2.1 (Pin_1), JB3.1 (Pin_1), JB4.1 (Pin_1), JB5.1 (Pin_1), JB6.1 (Pin_1), JB7.1 (Pin_1), JRST0.1 (Pin_1), JSRC0.1 (Pin_1); no longer JB0.6 (Pin_6), JB1.6 (Pin_6), JB2.6 (Pin_6), JB3.6 (Pin_6), JB4.6 (Pin_6), JB5.6 (Pin_6), JB6.6 (Pin_6), JB7.6 (Pin_6), JRST0.2 (Pin_2), JSRC0.6 (Pin_6)
- net LED-INT-IND: now also JB7.6 (Pin_6); no longer JB7.1 (Pin_1)
- net LED-SIG: now also JB0.5 (Pin_5); no longer JB0.2 (Pin_2)
- net RESET: now also JRST0.2 (Pin_2); no longer JRST0.1 (Pin_1)
- net ROW0: now also JB0.3 (Pin_3), JB1.3 (Pin_3), JB2.3 (Pin_3), JB3.3 (Pin_3), JSRC0.5 (Pin_5); no longer JB0.4 (Pin_4), JB1.4 (Pin_4), JB2.4 (Pin_4), JB3.4 (Pin_4), JSRC0.2 (Pin_2)
- net ROW1: now also JB4.3 (Pin_3), JB5.3 (Pin_3), JB6.3 (Pin_3), JB7.3 (Pin_3), JSRC0.6 (Pin_6); no longer JB4.4 (Pin_4), JB5.4 (Pin_4), JB6.4 (Pin_4), JB7.4 (Pin_4), JSRC0.1 (Pin_1)
- new net: JB1.6 (Pin_6), JB2.5 (Pin_5)
- new net: JB2.6 (Pin_6), JB3.5 (Pin_5)
- new net: JB5.6 (Pin_6), JB6.5 (Pin_5)
- new net: JB6.6 (Pin_6), JB7.5 (Pin_5)
- new net: JB0.6 (Pin_6), JB1.5 (Pin_5)
- new net: JB4.6 (Pin_6), JB5.5 (Pin_5)
- new net: JB3.6 (Pin_6), JB4.5 (Pin_5)
